File: HuskyA100_Nucleo_Shield.sch (KiCad schematic (older format))
At the start: 16 parts, among them CN10 HEADER_17x2, CN7 HEADER_10x2, CN8 HEADER_8x2, CN9 HEADER_15x2, J1 Conn_01x03, J2 Conn_01x03, J3 Conn_01x04, J4 Conn_01x04

Commit message: Fix #4 - added power led and authorship. Also made the capacitor pads to 'hand-solderable' for easier assembly
Parts:
- added D1: LED, LED_SMD:LED_PLCC-2, symbol Device:LED
- added R1: 66.5 Ohm, Resistor_SMD:R_1206_3216Metric_Pad1.42x1.75mm_HandSolder, symbol Device:R
- C1, C2, C3, C4, C5, C6, C7, C8: footprint Capacitor_SMD:C_2220_5650Metric -> Capacitor_SMD:C_2220_5650Metric_Pad1.97x5.40mm_HandSolder
Connections:
- net 5V: now also D1.2 (A)
- net GND: now also CN10.21, CN10.28, CN9.11, R1.1
- new net: D1.1 (K), R1.2
Changed lines of the file:
@@
 Text GLabel 2800 4050 2    50   Input ~ 0
 GND
-Text GLabel 5700 4600 2    50   Input ~ 0
+Text GLabel 4150 5000 0    50   Input ~ 0
 GND
 Text GLabel 7450 2200 2    50   Input ~ 0
@@
 F 0 "C1" H 3315 2396 50  0000 L CNN
 F 1 "0.01uF" H 3315 2305 50  0000 L CNN
-F 2 "Capacitor_SMD:C_2220_5650Metric" H 3238 2200 50  0001 C CNN
+F 2 "Capacitor_SMD:C_2220_5650Metric_Pad1.97x5.40mm_HandSolder" H 3238 2200 50  0001 C CNN
 F 3 "~" H 3200 2350 50  0001 C CNN
 	1    3200 2350
@@
 F 0 "C2" H 3865 2396 50  0000 L CNN
 F 1 "0.01uF" H 3865 2305 50  0000 L CNN
-F 2 "Capacitor_SMD:C_2220_5650Metric" H 3788 2200 50  0001 C CNN
+F 2 "Capacitor_SMD:C_2220_5650Metric_Pad1.97x5.40mm_HandSolder" H 3788 2200 50  0001 C CNN
 F 3 "~" H 3750 2350 50  0001 C CNN
 	1    3750 2350
@@
 F 0 "C3" H 4465 2396 50  0000 L CNN
 F 1 "0.01uF" H 4465 2305 50  0000 L CNN
-F 2 "Capacitor_SMD:C_2220_5650Metric" H 4388 2200 50  0001 C CNN
+F 2 "Capacitor_SMD:C_2220_5650Metric_Pad1.97x5.40mm_HandSolder" H 4388 2200 50  0001 C CNN
 F 3 "~" H 4350 2350 50  0001 C CNN
 	1    4350 2350
@@
 F 0 "C4" H 4965 2396 50  0000 L CNN
 F 1 "0.01uF" H 4965 2305 50  0000 L CNN
-F 2 "Capacitor_SMD:C_2220_5650Metric" H 4888 2200 50  0001 C CNN
+F 2 "Capacitor_SMD:C_2220_5650Metric_Pad1.97x5.40mm_HandSolder" H 4888 2200 50  0001 C CNN
 F 3 "~" H 4850 2350 50  0001 C CNN
 	1    4850 2350
@@
 F 0 "C5" H 5415 2396 50  0000 L CNN
 F 1 "0.1uF" H 5415 2305 50  0000 L CNN
-F 2 "Capacitor_SMD:C_2220_5650Metric" H 5338 2200 50  0001 C CNN
+F 2 "Capacitor_SMD:C_2220_5650Metric_Pad1.97x5.40mm_HandSolder" H 5338 2200 50  0001 C CNN
 F 3 "~" H 5300 2350 50  0001 C CNN
 	1    5300 2350
@@
 F 0 "C6" H 5865 2396 50  0000 L CNN
 F 1 "0.1uF" H 5865 2305 50  0000 L CNN
-F 2 "Capacitor_SMD:C_2220_5650Metric" H 5788 2200 50  0001 C CNN
+F 2 "Capacitor_SMD:C_2220_5650Metric_Pad1.97x5.40mm_HandSolder" H 5788 2200 50  0001 C CNN
 F 3 "~" H 5750 2350 50  0001 C CNN
 	1    5750 2350
@@
 F 0 "C7" H 6315 2396 50  0000 L CNN
 F 1 "0.1uF" H 6315 2305 50  0000 L CNN
-F 2 "Capacitor_SMD:C_2220_5650Metric" H 6238 2200 50  0001 C CNN
+F 2 "Capacitor_SMD:C_2220_5650Metric_Pad1.97x5.40mm_HandSolder" H 6238 2200 50  0001 C CNN
 F 3 "~" H 6200 2350 50  0001 C CNN
 	1    6200 2350
@@
 F 0 "C8" H 6765 2396 50  0000 L CNN
 F 1 "0.1uF" H 6765 2305 50  0000 L CNN
-F 2 "Capacitor_SMD:C_2220_5650Metric" H 6688 2200 50  0001 C CNN
+F 2 "Capacitor_SMD:C_2220_5650Metric_Pad1.97x5.40mm_HandSolder" H 6688 2200 50  0001 C CNN
 F 3 "~" H 6650 2350 50  0001 C CNN
 	1    6650 2350
@@
 Wire Wire Line
 	6650 2500 7450 2500
+Text GLabel 6800 3200 0    50   Input ~ 0
+5V
+Text GLabel 8000 3200 2    50   Input ~ 0
+GND
+$Comp
+L Device:LED D1
+U 1 1 5C67677D
+P 7100 3200
+F 0 "D1" H 7092 2945 50  0000 C CNN
+F 1 "LED" H 7092 3036 50  0000 C CNN
+F 2 "LED_SMD:LED_PLCC-2" H 7100 3200 50  0001 C CNN
+F 3 "~" H 7100 3200 50  0001 C CNN
+	1    7100 3200
+	-1   0    0    1
+$EndComp
+$Comp
+L Device:R R1
+U 1 1 5C676922
+P 7650 3200
+F 0 "R1" V 7443 3200 50  0000 C CNN
+F 1 "66.5 Ohm" V 7534 3200 50  0000 C CNN
+F 2 "Resistor_SMD:R_1206_3216Metric_Pad1.42x1.75mm_HandSolder" V 7580 3200 50  0001 C CNN
+F 3 "~" H 7650 3200 50  0001 C CNN
+	1    7650 3200
+	0    1    1    0
+$EndComp
+Wire Wire Line
+	7800 3200 8000 3200
+Wire Wire Line
+	7500 3200 7250 3200
+Wire Wire Line
+	6950 3200 6800 3200
+Text GLabel 5400 5400 0    50   Input ~ 0
+GND
+Text GLabel 5700 5700 2    50   Input ~ 0
+GND
+Text GLabel 5700 4600 2    50   Input ~ 0
+GND
 $EndSCHEMATC

Commit message: added a title, miscellaneous fixes changes
Connections:
- net 3.3V: now also J3.4 (Pin_4), J4.4 (Pin_4); no longer J3.3 (Pin_3), J4.3 (Pin_3)
- net GND: now also J1.1 (Pin_1), J2.1 (Pin_1), J3.3 (Pin_3), J4.3 (Pin_3); no longer J1.3 (Pin_3), J2.3 (Pin_3), J3.4 (Pin_4), J4.4 (Pin_4)
- net at CN7.1: now also J1.3 (Pin_3); no longer J1.1 (Pin_1)
- net at CN7.3: now also J2.3 (Pin_3); no longer J2.1 (Pin_1)
Changed lines of the file:
@@
 Text GLabel 4450 3800 2    50   Input ~ 0
 3.3V
+Text GLabel 2800 4050 2    50   Input ~ 0
+3.3V
+Text GLabel 3100 3400 2    50   Input ~ 0
+3.3V
+Text GLabel 5000 3450 2    50   Input ~ 0
+GND
+Text GLabel 5000 3350 2    50   Input ~ 0
+3.3V
+Text GLabel 3100 3300 2    50   Input ~ 0
+GND
 Text GLabel 2800 3950 2    50   Input ~ 0
-3.3V
-Text GLabel 3100 3300 2    50   Input ~ 0
-3.3V
-Text GLabel 5000 3250 2    50   Input ~ 0
-GND
-Text GLabel 5000 3350 2    50   Input ~ 0
-3.3V
-Text GLabel 3100 3400 2    50   Input ~ 0
-GND
-Text GLabel 2800 4050 2    50   Input ~ 0
 GND
 Text GLabel 4150 5000 0    50   Input ~ 0
@@
 Text GLabel 5000 2850 2    50   Input ~ 0
 3.3V
-Text GLabel 5000 2950 2    50   Input ~ 0
-GND
-Wire Wire Line
-	5000 2750 5300 2750
-Wire Wire Line
-	5300 2750 5300 3150
-Wire Wire Line
-	5300 3150 5400 3150
-Wire Wire Line
-	5000 3450 5300 3450
-Wire Wire Line
-	5300 3450 5300 3250
-Wire Wire Line
-	5300 3250 5400 3250
+Text GLabel 5000 2750 2    50   Input ~ 0
+GND
 Wire Wire Line
 	2950 2200 3200 2200
@@
 Text GLabel 5700 4600 2    50   Input ~ 0
 GND
+Wire Wire Line
+	5000 3150 5000 2950
+Wire Wire Line
+	5000 3150 5400 3150
+Wire Wire Line
+	5000 3250 5400 3250
 $EndSCHEMATC
